File: Buoy.kicad_pcb (KiCad board)
At the start: 4 copper layers, 150 x 110.8 mm, 144 parts, among them J1 Barrel_Jack_Switch, J10 Conn_01x05_Socket, J11 Screw_Terminal_01x02, J13 Conn_01x06_Socket, J14 Screw_Terminal_01x02, J2 Barrel_Jack_Switch, J3 Barrel_Jack_Switch, J4 Barrel_Jack_Switch, J5 Barrel_Jack_Switch, J6 Barrel_Jack_Switch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

Commit message: submitted for production
Parts:
- removed the . at (92.3, 46.1)
- added .: LOGO, Logos:CNPQ, F.Cu at (166.7, 131.9)
- added .: LOGO, Logos:CNPQ, B.Cu at (166.0, 132.0)
- added ?: MountingHole_2.2mm_M2_ISO14580, MountingHole:MountingHole_2.2mm_M2_ISO14580, F.Cu at (80.2, 136.6)
- added ?: MountingHole_2.2mm_M2_ISO14580, MountingHole:MountingHole_2.2mm_M2_ISO14580, F.Cu at (222.5, 43.8)
- added ?: MountingHole_2.2mm_M2_ISO14580, MountingHole:MountingHole_2.2mm_M2_ISO14580, F.Cu at (221.8, 136.4)
- added ?: MountingHole_2.2mm_M2_ISO14580, MountingHole:MountingHole_2.2mm_M2_ISO14580, F.Cu at (79.8, 43.8)
- added G***: LOGO, Logos:INEOF, F.Cu at (192.2, 134.3)
- added G***: LOGO, Logos:BoiasLivres, F.Cu at (139.2, 57.2)
- added G***: LOGO, Logos:INEOF, B.Cu at (192.2, 134.3)
- added G***: LOGO, Logos:BoiasLivres, B.Cu at (139.6, 57.2)
- C10, C16, C21, C22, C23, C24, C25, C26, C3, C6: footprint Capacitor_SMD:C_1210_3225Metric_Pad1.33x2.70mm_HandSolder -> Capacitor_SMD:C_0805_2012Metric_Pad1.18x1.45mm_HandSolder
- C15: footprint Capacitor_SMD:C_1206_3216Metric_Pad1.33x1.80mm_HandSolder -> Capacitor_SMD:C_0603_1608Metric_Pad1.08x0.95mm_HandSolder
- C35: footprint Capacitor_SMD:C_0201_0603Metric_Pad0.64x0.40mm_HandSolder -> Capacitor_SMD:C_0805_2012Metric_Pad1.18x1.45mm_HandSolder
- R19, R20: value 5.1k -> 1.7k
- moved TP17 13.0 mm to (198.2, 88.3)
- moved C26 7.39 mm to (203.8, 62.1)
- moved J14 7.00 mm to (213.0, 49.5)
- moved R28 6.83 mm to (209.4, 59.4)
- moved C25 6.06 mm to (203.8, 66.2)
- moved J8 5.50 mm to (207.2, 131.4)
- moved R27 5.39 mm to (209.4, 64.0)
- moved C24 4.88 mm to (203.8, 70.3)
- moved R26 4.15 mm to (209.5, 68.5)
- moved C23 3.75 mm to (203.7, 74.5)
- moved R23 2.80 mm to (209.8, 82.5)
- moved C22 2.65 mm to (203.7, 78.6)
- moved J13 2.05 mm to (218.8, 71.6)
- moved R24 1.81 mm to (209.7, 77.8)
- moved C15 1.63 mm to (142.0, 94.4)
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Routing:
- net Net-(U4-VC0): track 27.5 -> 18.7 mm
- net /Batman: track 74.6 -> 65.9 mm
- net Net-(J14-Pin_1): track 77.5 -> 70.6 mm
- net /Bat_in: track 249.1 -> 243.1 mm
- net Net-(J13-Pin_1): track 16.1 -> 12.0 mm
- net Net-(U4-VC1): track 23.9 -> 20.1 mm
- net Net-(J13-Pin_2): track 11.2 -> 7.77 mm
- net Net-(J13-Pin_3): track 12.2 -> 10.2 mm
- net Net-(U4-VC2): track 16.2 -> 14.3 mm
- net Net-(J13-Pin_5): track 11.8 -> 10.2 mm
- net Net-(J13-Pin_4): track 7.16 -> 6.17 mm
- net /3.4V: track 64.6 -> 63.7 mm
- net /Bat_out: track 72.6 -> 73.2 mm
- net PGND: track 85.9 -> 85.3 mm
- net Net-(U4-VC3): track 14.8 -> 14.2 mm
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- added copper zone on In2.Cu, net PGND
