File: Buoy.kicad_sch (KiCad schematic)
At the start: 119 parts, among them J1 Barrel_Jack, J10 Conn_01x03_Pin, J2 Barrel_Jack, J3 Barrel_Jack, J4 Barrel_Jack, J5 Barrel_Jack, J6 Barrel_Jack, J7 Screw_Terminal_01x02, J8 Screw_Terminal_01x02, J9 Conn_01x03_Pin, Q1 AO3401A, Q2 AO3401A, Q3 BSS138, Q4 SI7288DP-T1-GE3, Q5 2N7002, Q6 AO3401A, Q7 BSS138, Q8 AO3401A, SW1 SW_Push_DPDT, U1 LM324, U2 BQ24650RVAR, U3 INA138, U4 SN74LVC1G74DCTR, U5 TPS62822DLC, U6 AP2112K-3.3

Commit message: version 1 for consultation
Parts:
- removed C13: 8.2nF, Capacitor_SMD:C_0603_1608Metric_Pad1.08x0.95mm_HandSolder, symbol Device:C
- removed C16: 1uF, Capacitor_SMD:C_1210_3225Metric_Pad1.33x2.70mm_HandSolder, symbol Device:C
- removed C19: 1nF, Capacitor_SMD:C_1210_3225Metric_Pad1.33x2.70mm_HandSolder, symbol Device:C
- removed C20: 220pF, Capacitor_SMD:C_0603_1608Metric_Pad1.08x0.95mm_HandSolder, symbol Device:C
- removed C27, C28: 330uF, Capacitor_SMD:C_Elec_10x10.2, symbol Device:C_Polarized_US
- removed C31(C1ondatasheet)1: 2.2u, symbol Device:C
- removed D4: LED, LTST-C190GKT:LEDC1608X35N, symbol Device:LED
- removed J1, J2, J3, J4, J5, J6: Barrel_Jack, Connector_BarrelJack:BarrelJack_Wuerth_6941xx301002, symbol Connector:Barrel_Jack
- removed J10: Conn_01x03_Pin, symbol Connector:Conn_01x03_Pin
- removed Q1, Q2, Q6, Q8: AO3401A, Package_TO_SOT_SMD:SOT-23, symbol Transistor_FET:AO3401A
- removed Q3, Q7: BSS138, Package_TO_SOT_SMD:SOT-23, symbol Transistor_FET:BSS138
- removed Q5: 2N7002, 2N7002_:SOT23, symbol Transistor_FET:2N7002
- removed R11: 100k, Resistor_SMD:R_0402_1005Metric_Pad0.72x0.64mm_HandSolder, symbol Device:R_US
- removed R4: 10k, Resistor_SMD:R_0805_2012Metric_Pad1.20x1.40mm_HandSolder, symbol Device:R_US
- removed R5: 2, Resistor_SMD:R_2512_6332Metric_Pad1.40x3.35mm_HandSolder, symbol Device:R_US
- removed RT12: 55k, symbol Device:R_US
- removed RT9: 6.6k, symbol Device:R_US
- removed SW1: SW_Push_DPDT, Switch SK22D15L5:SK22D15L5, symbol Switch:SW_Push_DPDT
- removed TP12, TP14, TP18, TP2: TestPoint, symbol Connector:TestPoint
- removed U1: LM324, LM324DT:SOIC127P600X175-14N, symbol Amplifier_Operational:LM324
- removed U4: SN74LVC1G74DCTR, SN74LVC1G74DCTR:SOP65P400X130-8N, symbol SN74LVC1G74DCTR:SN74LVC1G74DCTR
- removed U5: TPS62822DLC, TPS62822DLCR:DLC0008A, symbol Regulator_Switching:TPS62822DLC
- added C22, C25, C26, C27, C28: 1uF, Capacitor_SMD:C_1210_3225Metric_Pad1.33x2.70mm_HandSolder, symbol Device:C
- added C31, C32: 100nF, Capacitor_SMD:C_0805_2012Metric_Pad1.18x1.45mm_HandSolder, symbol Device:C
- added C33: 4.7uF, Capacitor_SMD:C_0805_2012Metric_Pad1.18x1.45mm_HandSolder, symbol Device:C
- added C34, C36: 22uF, Capacitor_SMD:C_0805_2012Metric_Pad1.18x1.45mm_HandSolder, symbol Device:C
- added C35: 100nF, Capacitor_SMD:C_0201_0603Metric_Pad0.64x0.40mm_HandSolder, symbol Device:C
- added CBJ1, CBJ2, CBJ3, CBJ4, CBJ5, CBJ6: 2.2uF, Capacitor_SMD:C_1210_3225Metric_Pad1.33x2.70mm_HandSolder, symbol Device:C
- added D10: 1N4148, Diode_SMD:D_SOD-323_HandSoldering, symbol Diode:1N4148
- added D4, D5, D7, D8, D9: PDS1040L-13, PDS1040L-13_solar:DIO_PDS1040L-13, symbol PDS1040L-13:PDS1040L-13
- added J1, J2, J3, J4, J5, J6: Barrel_Jack_Switch, Barrel_Jack:XKB_DC-005-5A-2.0, symbol Connector:Barrel_Jack_Switch
- added J10: Conn_01x05_Socket, Connector_PinHeader_2.54mm:PinHeader_1x05_P2.54mm_Vertical_SMD_Pin1Right, symbol Connector:Conn_01x05_Socket
- added J11, J14: Screw_Terminal_01x02, Screw_Terminal:CONN_1729128_PXC, symbol Connector:Screw_Terminal_01x02
- added J13: Conn_01x06_Socket, Connector_PinHeader_2.54mm:PinHeader_1x06_P2.54mm_Vertical_SMD_Pin1Right, symbol Connector:Conn_01x06_Socket
- added Q1: SI7288DP-T1-GE3, SI7288DP:TRANS_SI7288DP-T1-GE3, symbol SI7288DP-T1-GE3:SI7288DP-T1-GE3
- added Q2: BS250, B2250MOSFET:SOT95P240X110-3N, symbol Transistor_FET:BS250
- added R12: 0.1, Resistor_SMD:R_2010_5025Metric_Pad1.40x2.65mm_HandSolder, symbol Device:R_US
- added R20: 5.1k, Resistor_SMD:R_1206_3216Metric_Pad1.30x1.75mm_HandSolder, symbol Device:R_US
- added R21: 10k, My_Passive:R_0402_1005Metric_Pad0.72x0.64mm_HandSolder, symbol Device:R_US
- added R30: 1M, Resistor_SMD:R_1206_3216Metric_Pad1.30x1.75mm_HandSolder, symbol Device:R_US
- added R34, R35: 100, Resistor_SMD:R_1210_3225Metric_Pad1.30x2.65mm_HandSolder, symbol Device:R_US
- added R36: 30k, Resistor_SMD:R_0603_1608Metric_Pad0.98x0.95mm_HandSolder, symbol Device:R_US
- added R37: 7.5k, My_Passive:R_0402_1005Metric_Pad0.72x0.64mm_HandSolder, symbol Device:R_US
- added RBJ1, RBJ2, RBJ3, RBJ4, RBJ5, RBJ6: 2, Resistor_SMD:R_2512_6332Metric_Pad1.40x3.35mm_HandSolder, symbol Device:R_US
- added SW1, SW2, SW3, SW4: SW_SPDT, Slide_Switch:SW-SPDT-SW, symbol Switch:SW_SPDT
- added TH1: Thermistor_NTC_US, Thermistor:THRMC1005X55N, symbol Device:Thermistor_NTC_US
- added U1: OPA340NA, Package_TO_SOT_SMD:SOT-23-5, symbol Amplifier_Operational:OPA340NA
- added U4: BQ76920PW, Package_SO:TSSOP-20_4.4x6.5mm_P0.65mm, symbol Battery_Management:BQ76920PW
- added U5: TPS564257DRLR, 3.4_Stepdown:TPS564242DRLR_TEX, symbol TPS564242DRLR:TPS564257DRLR
- C1: value 220pF -> 10nF; footprint Capacitor_SMD:C_0201_0603Metric_Pad0.64x0.40mm_HandSolder -> Capacitor_SMD:C_0805_2012Metric_Pad1.18x1.45mm_HandSolder
- C11, C21: value 100nF -> 1uF; footprint Capacitor_SMD:C_0805_2012Metric_Pad1.18x1.45mm_HandSolder -> Capacitor_SMD:C_1210_3225Metric_Pad1.33x2.70mm_HandSolder
- C12: value 4.7uF -> 100nF; footprint Capacitor_SMD:C_0805_2012Metric_Pad1.18x1.45mm_HandSolder -> Capacitor_SMD:C_0603_1608Metric_Pad1.08x0.95mm_HandSolder
- C17: value 1uF -> 22uF
- C18: value 100nF -> 10pF; footprint Capacitor_SMD:C_0805_2012Metric_Pad1.18x1.45mm_HandSolder -> My_Passive:C_0402_1005Metric_Pad0.74x0.62mm_HandSolder
- C23: value 120pF -> 1uF; footprint Capacitor_SMD:C_01005_0402Metric_Pad0.57x0.30mm_HandSolder -> Capacitor_SMD:C_1210_3225Metric_Pad1.33x2.70mm_HandSolder
- C24: value 22uF -> 1uF; footprint Capacitor_SMD:C_1206_3216Metric_Pad1.33x1.80mm_HandSolder -> Capacitor_SMD:C_1210_3225Metric_Pad1.33x2.70mm_HandSolder
- C29: value 33pF -> 1uF; footprint Capacitor_SMD:C_0805_2012Metric_Pad1.18x1.45mm_HandSolder -> Capacitor_SMD:C_1210_3225Metric_Pad1.33x2.70mm_HandSolder
- C30: value 10pF -> 100nF
- C9: value 10nF -> 8.2nF; footprint Capacitor_SMD:C_0805_2012Metric_Pad1.18x1.45mm_HandSolder -> Capacitor_SMD:C_0603_1608Metric_Pad1.08x0.95mm_HandSolder
- D1: footprint PDS1040L-13:DIO_PDS1040L-13 -> PDS1040L-13_solar:DIO_PDS1040L-13
- D2: value yellow -> LED; footprint LTST-C190GKT:LEDC1608X35N -> LED:LEDC1608X35N
- D3: value green -> LED; footprint LTST-C190GKT:LEDC1608X35N -> LED:LEDC1608X35N
- J7, J8: footprint Screw_Term_1x2:CONN_1729128_PXC -> Screw_Terminal:CONN_1729128_PXC
- J9: footprint (none) -> Connector_PinHeader_2.54mm:PinHeader_1x03_P2.54mm_Vertical_SMD_Pin1Right
- L1: footprint Inductor_SMD:L_Koher_MDA1350_13.5x12.6mm_1 -> L_MPPT:L_Koher_MDA1350_13.5x12.6mm_1
- L2: value 0.47uH -> 1.5uH; footprint IHLP-2525CZ-01:2525 -> L_3.4:L_Vishay_IHLP-2020
- Q4: footprint SI7288DP-T1-GE3:TRANS_SI7288DP-T1-GE3 -> SI7288DP:TRANS_SI7288DP-T1-GE3
- R1: value 0 -> 5.1k; footprint (none) -> Resistor_SMD:R_1206_3216Metric_Pad1.30x1.75mm_HandSolder
- R10: footprint (none) -> My_Passive:R_0402_1005Metric_Pad0.72x0.64mm_HandSolder
- R11: renamed from R30; footprint (none) -> Resistor_SMD:R_1206_3216Metric_Pad1.30x1.75mm_HandSolder
- R14: value 0.1 -> 24.9k; footprint (none) -> My_Passive:R_0402_1005Metric_Pad0.72x0.64mm_HandSolder
- R16: value 33k -> 53.6k; footprint (none) -> My_Passive:R_0402_1005Metric_Pad0.72x0.64mm_HandSolder
- R17: value 1k -> 30k; footprint (none) -> Resistor_SMD:R_0603_1608Metric_Pad0.98x0.95mm_HandSolder
- R18: value 1k -> 100; footprint (none) -> Resistor_SMD:R_1210_3225Metric_Pad1.30x2.65mm_HandSolder
- R19: value 1k -> 5.1k; footprint (none) -> Resistor_SMD:R_1206_3216Metric_Pad1.30x1.75mm_HandSolder
- R2: value 220k -> 100k; footprint Resistor_SMD:R_0402_1005Metric_Pad0.72x0.64mm_HandSolder -> My_Passive:R_0402_1005Metric_Pad0.72x0.64mm_HandSolder
- R22: value 390 -> 140k; footprint (none) -> Resistor_SMD:R_0805_2012Metric_Pad1.20x1.40mm_HandSolder
- R23: value 220k -> 100; footprint (none) -> Resistor_SMD:R_1210_3225Metric_Pad1.30x2.65mm_HandSolder
- R24: value 10 -> 100; footprint (none) -> Resistor_SMD:R_1210_3225Metric_Pad1.30x2.65mm_HandSolder
- R25, R33: value 10k -> 100; footprint Resistor_SMD:R_0805_2012Metric_Pad1.20x1.40mm_HandSolder -> Resistor_SMD:R_1210_3225Metric_Pad1.30x2.65mm_HandSolder
- R26: value 22k -> 100; footprint (none) -> Resistor_SMD:R_1210_3225Metric_Pad1.30x2.65mm_HandSolder
- R27: value 0 -> 100; footprint (none) -> Resistor_SMD:R_1210_3225Metric_Pad1.30x2.65mm_HandSolder
- R28: value 460k -> 100; footprint (none) -> Resistor_SMD:R_1210_3225Metric_Pad1.30x2.65mm_HandSolder
- R29: value 100k -> 20m; footprint (none) -> Resistor_SMD:R_2010_5025Metric_Pad1.40x2.65mm_HandSolder
- R3: value 22k -> 10k; footprint Resistor_SMD:R_0603_1608Metric_Pad0.98x0.95mm_HandSolder -> Resistor_SMD:R_0805_2012Metric_Pad1.20x1.40mm_HandSolder
- R31: value 10 -> 1M; footprint (none) -> Resistor_SMD:R_1206_3216Metric_Pad1.30x1.75mm_HandSolder
- R32: value 0 -> 1M; footprint (none) -> Resistor_SMD:R_1206_3216Metric_Pad1.30x1.75mm_HandSolder
- R9: footprint Resistor_SMD:R_0402_1005Metric_Pad0.72x0.64mm_HandSolder -> My_Passive:R_0402_1005Metric_Pad0.72x0.64mm_HandSolder
- TP1, TP10, TP11, TP13, TP15, TP16, TP17, TP19, TP20, TP3, TP4, TP5, TP6, TP7, TP8, TP9: footprint (none) -> TestpointMINE:TestPoint_Pad_1.0x1.0mm
- U2: footprint BQ24650RVAT:QFN50P350X350X100-17N -> BQ24650:QFN50P350X350X100-17N; Purchase-URL https://www.snapeda.com/api/url_track_click_mouser/?unipart_id=281663&manufacturer=Texas Instruments&part_name=BQ24650RVAT&search_term=None -> https://www.snapeda.com/api/url_track_click_mouser/?unipart_id=281663&manufacturer=Texas Instruments&part_name=BQ24650RVAT&search_term=bq24650
- U3: footprint INA138NA_3K:SOT95P280X145-5N -> INA138:SOT95P280X145-5N
- U6: footprint AP2112K-3.3TRG1:SOT95P285X140-5N -> 3.3_LDO:SOT95P285X140-5N
- renumbered C31 to C13, C16(C3ondatasheet)1 to C16, C25 to C19, C26 to C20, R20 to R4, R21 to R5
Connections:
- net 3.4V: now also C18.1, C19.1, R22.1, U6.1 (VIN), U6.3 (EN), C34.1, C35.1, C36.1, J11.1 (Pin_1), R21.2; no longer C11.1, C23.1, C24.1, R14.1, R28.1, TP6.1, U3.3 (+), U3.5 (V+)
- net ADC VBAT: now also C1.1, R10.1, R2.2, TP3.1; no longer C9.1, R10.2, TP5.1
- net ADC current: now also C11.1, R18.2, TP7.1; no longer R17.2, TP11.1
- net TS: now also R1.1, TP10.1, R37.1
- net VREF: now also R1.2
- net at R24.1: now also C21.2, C22.1, U4.13 (VC4)
- net at R18.1: now also TP8.1, U1.1, U1.4 (-); no longer TP10.1
- net at R19.2: now also J10.4 (Pin_4), U4.4 (SDA)
- net at R26.2: now also J13.3 (Pin_3)
- net at R27.1: now also C24.2, R3.1, C25.1, U4.16 (VC1); no longer TP4.1
- net PV_connection: now reaches D1.1, D1.2, R6.1
- net PV_connection: now also D4.1, D4.2, D5.1, D5.2, D7.1, D7.2, D8.1, D8.2, D9.1, D9.2, J1.1, J2.1, J3.1, J4.1, J5.1, J6.1, RBJ1.1, RBJ2.1, RBJ3.1, RBJ4.1, RBJ5.1, RBJ6.1; no longer R8.1, TP19.1
- net Batman: now reaches TP17.1
- net Batman: now also R23.2, R33.1, C28.1, J13.6 (Pin_6), SW3.3 (C), SW4.3 (C), U4.9 (REGSRC); no longer R31.2
- net Bat_out: now reaches C2.1, R2.1
- net Bat_out: now also J8.1 (Pin_1), TP4.1, U3.3 (+), U3.5 (V+), R12.1, SW4.2 (B); no longer C1.1, R1.2
- net at C17.1: now also C12.1, R16.1, TP5.1, U3.4 (-), R12.2, U1.5 (V+), U5.1 (VIN); no longer R18.2
- net V_solar_out: now reaches C13.1, Q4.7_8_9, R11.1
- net V_solar_out: now also R8.1, TP19.1, SW1.3 (C); no longer D1.3
- net at C3.1, R6.2, R7.1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: now also TP11.1
- net Power_out: now reaches C14.1, L1.2, R6_SR1.1, TP15.1, U2.10 (SRP)
- net PH: now reaches C5.2, L1.1, Q4.1, Q4.5_6_10, TP13.1, U2.14 (PH)
- net at R31.1: now also R32.2, D10.1 (K), Q1.4
- net at R17.1: now also R16.2, U5.5 (EN); no longer TP9.1
- net at L2.1: now also U5.2 (SW)
- net at R22.2: now also C18.2, R36.1, U5.6 (FB)
- net at R3.2: now also J10.1 (Pin_1), TH1.1, U4.6 (TS1)
- net at J7.1 (Pin_1): now also C20.1, TP1.1, U6.5 (VOUT)
- net GNDA renamed PGND
- net PGND: now also C2.2, R10.2, R14.2, R17.2, R31.2, C25.2, C26.1, C27.2, C28.2, C31.2, C32.1, C33.2, C34.2, C35.2, C36.2, CBJ1.2, CBJ2.2, CBJ3.2, CBJ4.2, CBJ5.2, CBJ6.2, J1.2, J1.3, J11.2 (Pin_2), J2.2, J2.3, J3.2, J3.3, J4.2, J4.3, J5.2, J5.3, J6.2, J6.3, Q1.3, Q2.2 (G), R36.2, R37.2, SW2.3 (C), TH1.2, U1.2 (V-), U4.3 (VSS), U5.3 (GND); no longer C18.2, C20.1, C24.2, C30.2, R16.2, R25.2, R29.2, R33.2, TP1.1, U6.5 (VOUT)
- net Vbat1 renamed Bat_in
- net Bat_in: now also J14.2 (Pin_2), SW3.2 (B)
- removed net Vbat2: C12.1, R10.1, R32.1
- new net: C23.2, C24.1, R26.1, U4.15 (VC2)
- new net: C21.1, R23.1, U4.12 (VC5)
- new net: J10.2 (Pin_2), U4.20 (ALERT)
- new net: J10.3 (Pin_3), R20.2, U4.5 (SCL)
- new net: C33.1, J10.5 (Pin_5), R19.1, R20.1, U4.8 (REGOUT)
- new net: CBJ4.1, RBJ4.2
- new net: Q1.5_6_10, Q1.7_8_9
- new net: Q1.1, R29.2, R30.2, R35.2
- new net: Q1.2, R30.1, U4.1 (DSG)
- new net: CBJ2.1, RBJ2.2
- new net: C9.1, R14.1, TP6.1, U1.3 (+), U3.1
- new net: CBJ5.1, RBJ5.2
- new net: C29.1, R33.2, U4.10 (BAT)
- new net: CBJ3.1, RBJ3.2
- new net: CBJ1.1, RBJ1.2
- new net: C26.2, R28.1, U4.17 (VC0)
- new net: J13.1 (Pin_1), R28.2
- new net: Q2.1 (D), U4.2 (CHG)
- new net: D10.2 (A), Q2.3 (S), R32.1
- new net: R29.1, R34.2, SW2.1 (A)
- new net: J14.1 (Pin_1), SW2.2 (B)
- new net: C22.2, C23.1, R25.1, U4.14 (VC3)
- new net: J13.4 (Pin_4), R25.2
- new net: CBJ6.1, RBJ6.2
- new net: C27.1, U4.7 (CAP1)
- new net: R21.1, U5.4 (PG)
- new net: C30.2, C32.2, R34.1, U4.18 (SRP)
- new net: J13.5 (Pin_5), R24.2
- new net: J13.2 (Pin_2), R27.2
- new net: C30.1, C31.1, R35.1, U4.19 (SRN)
- new net Non-Batman: SW3.1 (A), SW4.1 (A)
- new net V_solar_in: D1.3, D4.3, D5.3, D7.3, D8.3, D9.3, SW1.2 (B), TP9.1
- no-connect marks 0 -> 2
Other:
- company: (none) -> LabECO
- title: MCU -> Solar harvesting and voltage regulation
- moved on the sheet: C10, C13, C14, C15, C16, C19, C20, C3, C4, C5, C6, C7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

Commit message: submitted for production
Parts:
- C10, C16, C21, C22, C23, C24, C25, C26, C3, C6: footprint Capacitor_SMD:C_1210_3225Metric_Pad1.33x2.70mm_HandSolder -> Capacitor_SMD:C_0805_2012Metric_Pad1.18x1.45mm_HandSolder
- C15: footprint Capacitor_SMD:C_1206_3216Metric_Pad1.33x1.80mm_HandSolder -> Capacitor_SMD:C_0603_1608Metric_Pad1.08x0.95mm_HandSolder
- C35: footprint Capacitor_SMD:C_0201_0603Metric_Pad0.64x0.40mm_HandSolder -> Capacitor_SMD:C_0805_2012Metric_Pad1.18x1.45mm_HandSolder
- R19, R20: value 5.1k -> 1.7k
Connections:
- no-connect marks 2 -> 1
Changed lines of the file:
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@@
   )
   (no_connect (at 109.22 130.81))
-  (no_connect (at 101.6 148.59))
   (wire (pts (xy 300.99 157.48) (xy 300.99 156.21))
     (stroke (width 0) (type default))
@@
       (effects (font (size 1.27 1.27)) (justify left))
     )
-    (property "Footprint" "Capacitor_SMD:C_1210_3225Metric_Pad1.33x2.70mm_HandSolder" (at 458.1652 88.9 0)
+    (property "Footprint" "Capacitor_SMD:C_0805_2012Metric_Pad1.18x1.45mm_HandSolder" (at 458.1652 88.9 0)
       (effects (font (size 1.27 1.27)) hide)
     )
@@
       (effects (font (size 1.27 1.27)) (justify left))
     )
-    (property "Footprint" "Capacitor_SMD:C_1210_3225Metric_Pad1.33x2.70mm_HandSolder" (at 458.1652 58.42 0)
+    (property "Footprint" "Capacitor_SMD:C_0805_2012Metric_Pad1.18x1.45mm_HandSolder" (at 458.1652 58.42 0)
       (effects (font (size 1.27 1.27)) hide)
     )
@@
       (effects (font (size 1.27 1.27)) (justify left))
     )
-    (property "Footprint" "Capacitor_SMD:C_1206_3216Metric_Pad1.33x1.80mm_HandSolder" (at 378.1552 140.97 0)
+    (property "Footprint" "Capacitor_SMD:C_0603_1608Metric_Pad1.08x0.95mm_HandSolder" (at 378.1552 140.97 0)
       (effects (font (size 1.27 1.27)) hide)
     )
@@
       (effects (font (size 1.27 1.27)) (justify left))
     )
-    (property "Footprint" "Capacitor_SMD:C_1210_3225Metric_Pad1.33x2.70mm_HandSolder" (at 232.1052 157.48 0)
+    (property "Footprint" "Capacitor_SMD:C_0805_2012Metric_Pad1.18x1.45mm_HandSolder" (at 232.1052 157.48 0)
       (effects (font (size 1.27 1.27)) hide)
     )
@@
       (effects (font (size 1.27 1.27)) (justify left))
     )
-    (property "Footprint" "Capacitor_SMD:C_1210_3225Metric_Pad1.33x2.70mm_HandSolder" (at 239.7252 138.43 0)
+    (property "Footprint" "Capacitor_SMD:C_0805_2012Metric_Pad1.18x1.45mm_HandSolder" (at 239.7252 138.43 0)
       (effects (font (size 1.27 1.27)) hide)
     )
@@
       (effects (font (size 1.27 1.27)) (justify left))
     )
-    (property "Footprint" "Capacitor_SMD:C_0201_0603Metric_Pad0.64x0.40mm_HandSolder" (at 374.3452 314.96 0)
+    (property "Footprint" "Capacitor_SMD:C_0805_2012Metric_Pad1.18x1.45mm_HandSolder" (at 374.3452 314.96 0)
       (effects (font (size 1.27 1.27)) hide)
     )
@@
       (effects (font (size 1.27 1.27)) (justify left))
     )
-    (property "Footprint" "Capacitor_SMD:C_1210_3225Metric_Pad1.33x2.70mm_HandSolder" (at 458.1652 68.58 0)
+    (property "Footprint" "Capacitor_SMD:C_0805_2012Metric_Pad1.18x1.45mm_HandSolder" (at 458.1652 68.58 0)
       (effects (font (size 1.27 1.27)) hide)
     )
@@
       (effects (font (size 1.27 1.27)) (justify left))
     )
-    (property "Footprint" "Capacitor_SMD:C_1210_3225Metric_Pad1.33x2.70mm_HandSolder" (at 239.7252 119.38 0)
+    (property "Footprint" "Capacitor_SMD:C_0805_2012Metric_Pad1.18x1.45mm_HandSolder" (at 239.7252 119.38 0)
       (effects (font (size 1.27 1.27)) hide)
     )
@@
       (effects (font (size 1.27 1.27)) (justify left))
     )
-    (property "Footprint" "Capacitor_SMD:C_1210_3225Metric_Pad1.33x2.70mm_HandSolder" (at 303.2252 86.36 0)
+    (property "Footprint" "Capacitor_SMD:C_0805_2012Metric_Pad1.18x1.45mm_HandSolder" (at 303.2252 86.36 0)
       (effects (font (size 1.27 1.27)) hide)
     )
@@
       (effects (font (size 1.27 1.27)) (justify left))
     )
-    (property "Footprint" "Capacitor_SMD:C_1210_3225Metric_Pad1.33x2.70mm_HandSolder" (at 458.1652 109.22 0)
+    (property "Footprint" "Capacitor_SMD:C_0805_2012Metric_Pad1.18x1.45mm_HandSolder" (at 458.1652 109.22 0)
       (effects (font (size 1.27 1.27)) hide)
     )
@@
       (effects (font (size 1.27 1.27)) (justify left))
     )
-    (property "Footprint" "Capacitor_SMD:C_1210_3225Metric_Pad1.33x2.70mm_HandSolder" (at 458.1652 100.33 0)
+    (property "Footprint" "Capacitor_SMD:C_0805_2012Metric_Pad1.18x1.45mm_HandSolder" (at 458.1652 100.33 0)
       (effects (font (size 1.27 1.27)) hide)
     )
@@
       (effects (font (size 1.27 1.27)) (justify left))
     )
-    (property "Value" "5.1k" (at 408.94 58.42 0)
+    (property "Value" "1.7k" (at 408.94 58.42 0)
       (effects (font (size 1.27 1.27)) (justify left))
     )
@@
       (effects (font (size 1.27 1.27)) (justify left))
     )
-    (property "Value" "5.1k" (at 400.05 59.69 0)
+    (property "Value" "1.7k" (at 400.05 59.69 0)
       (effects (font (size 1.27 1.27)) (justify left))
     )
@@
       (effects (font (size 1.27 1.27)) (justify left))
     )
-    (property "Footprint" "Capacitor_SMD:C_1210_3225Metric_Pad1.33x2.70mm_HandSolder" (at 458.1652 78.74 0)
+    (property "Footprint" "Capacitor_SMD:C_0805_2012Metric_Pad1.18x1.45mm_HandSolder" (at 458.1652 78.74 0)
       (effects (font (size 1.27 1.27)) hide)
     )
